File: Hard/Idiotbox.sch (KiCad schematic (older format))
At the start: 46 parts

Commit message: Anottate
Parts:
- added J2, J4, J6: Conn_01x01_Female, symbol Connector:Conn_01x01_Female
- gave numbers to parts that had none: 43
- renumbered BASS to BASS1, GAIN to GAIN1, TREBLE to TREBLE1
Connections:
- net GND: now also J2.1 (Pin_1), J4.1 (Pin_1), J6.1 (Pin_1)
